File: hardware/kicad/ch375_board.kicad_sch (KiCad schematic)
At the start: 9 parts, among them IC1 ATF22V10C, J1 Conn_02x32_Odd_Even, J2 Conn_02x08_Odd_Even

Commit message: hardware: Updated the PCB design now that I actually understand how to do autovector interrupts!
Connections:
- net A1: now also IC1.1 (I1/CLK)
- net A12: now also IC1.4 (I4/PD); no longer IC1.2 (I2)
- net A13: now also IC1.5 (I5); no longer IC1.3 (I3)
- net A14: now also IC1.6 (I6); no longer IC1.4 (I4/PD)
- net A15: now also IC1.7 (I7); no longer IC1.5 (I5)
- net A16: now also IC1.8 (I8); no longer IC1.6 (I6)
- net A17: now also IC1.9 (I9); no longer IC1.7 (I7)
- net A18: now also IC1.10 (I10); no longer IC1.8 (I8)
- net A19: now also IC1.11 (I11); no longer IC1.9 (I9)
- net A2: now also IC1.2 (I2)
- net A3: now also IC1.3 (I3)
- net AS: now also IC1.18 (IO5); no longer IC1.16 (IO3)
- net CLK: no longer IC1.1 (I1/CLK)
- net DTACK: now also IC1.17 (I04); no longer IC1.22 (IO9)
- net FC0: now also IC1.21 (IO8)
- net FC1: now also IC1.20 (IO7)
- net FC2: now also IC1.19 (IO6)
- net IOSEL: now also IC1.22 (IO9); no longer IC1.11 (I11)
- net IRQ3: no longer IC1.19 (IO6)
- net IRQ5: now also J2.9 (Pin_9)
- net LDS: no longer IC1.15 (IO2)
- net R~{W}: now also IC1.16 (IO3); no longer IC1.14 (IO1)
- net VMA: no longer IC1.10 (I10)
- net W~{R}: now also IC1.15 (IO2); no longer IC1.20 (IO7)
- net ~{CHCS}: now also IC1.14 (IO1); no longer IC1.21 (IO8)
- net INT: no longer names the net of IC1.13 (I13)
- net INT: no longer J2.9 (Pin_9)
- no-connect marks 2 -> 1
Other:
- title: (none) -> CH375 and RAM Expansion Board
