File: hardware/kicad/expansion_ram_sch.kicad_sch (KiCad schematic)
At the start: 5 parts, among them IC2 ATF22V10C, U1 AS6C4008-55PCN, U2 AS6C4008-55PCN, U3 74HCT161, U4 74LS283

Commit message: hardware: Updated the PCB design now that I actually understand how to do autovector interrupts!
Connections:
- net A12: now also IC2.4 (I4/PD); no longer IC2.2 (I2)
- net A13: now also IC2.5 (I5); no longer IC2.3 (I3)
- net A14: now also IC2.6 (I6); no longer IC2.4 (I4/PD)
- net A15: now also IC2.7 (I7); no longer IC2.5 (I5)
- net A16: now also IC2.8 (I8); no longer IC2.6 (I6)
- net A17: now also IC2.9 (I9); no longer IC2.7 (I7)
- net A18: now also IC2.10 (I10); no longer IC2.8 (I8)
- net A19: now also IC2.11 (I11); no longer IC2.9 (I9)
- net AS: now also IC2.18 (IO5); no longer IC2.16 (IO3)
- net CLK: no longer IC2.1 (I1/CLK)
- net EXPSEL: now also IC2.21 (IO8); no longer IC2.11 (I11)
- net IOSEL: now also IC2.22 (IO9); no longer IC2.10 (I10)
- net LDS: now also IC2.19 (IO6); no longer IC2.15 (IO2)
- net R~{W}: now also IC2.16 (IO3); no longer IC2.13 (I13)
- net UDS: now also IC2.20 (IO7); no longer IC2.14 (IO1)
- net ~{BASESEL}: now also IC2.23 (IO10); no longer IC2.19 (IO6)
- net ~{ERAM1}: now also IC2.14 (IO1); no longer IC2.18 (IO5)
- net ~{ORAM1}: now also IC2.15 (IO2); no longer IC2.17 (I04)
- new net DTACK: IC2.17 (I04)
Other:
- title: (none) -> CH375 and RAM Expansion Board
